Commit message: Update line.xacro

File: line_description/urdf/line.xacro (robot description, xacro)
@@ -108,5 +108,5 @@
   <parent link="base_link"/>
   <child link="wheel2_1"/>
-  <axis xyz="0.0 -1.0 0.0"/>
+  <axis xyz="0.0 1.0 0.0"/>
 </joint>
 <joint name="Rev2" type="continuous">
@@ -114,5 +114,5 @@
   <parent link="base_link"/>
   <child link="wheel1_1"/>
-  <axis xyz="0.0 -1.0 0.0"/>
+  <axis xyz="0.0 1.0 0.0"/>
 </joint>
 <joint name="Rigid3" type="fixed">
